Commit message: gmapping - amcl -movebase

File: turtlebot3/turtlebot3_description/urdf/agv.urdf.xacro (robot description, xacro)
@@ -11,5 +11,5 @@
   <link name="base_link">
     <visual>
-      <origin xyz="-0.064 0 0.0" rpy="0 0 0"/>
+      <origin xyz="0.0 0 0.0" rpy="0 0 0"/>
       <geometry>
         <!-- <mesh filename="package://turtlebot3_description/meshes/bases/waffle_pi_base.stl" scale="0.001 0.001 0.001"/> -->
@@ -19,5 +19,5 @@
     </visual>
     <collision>
-      <origin xyz="-0.064 0 0.047" rpy="0 0 0"/>
+      <origin xyz="0.0 0 0.047" rpy="0 0 0"/>
       <geometry>
         <box size="0.266 0.266 0.094"/>
@@ -26,8 +26,8 @@
     <inertial>
       <origin xyz="0 0 0" rpy="0 0 0"/>
-      <mass value="1.3729096e+00"/>
-      <inertia ixx="8.7002718e-03" ixy="-4.7576583e-05" ixz="1.1160499e-04"
-               iyy="8.6195418e-03" iyz="-3.5422299e-06"
-               izz="1.4612727e-02" />
+      <mass value="16"/>
+      <inertia ixx="1" ixy="0" ixz="0"
+               iyy="1" iyz="0"
+               izz="1" />
     </inertial>
   </link>
@@ -35,9 +35,9 @@
     <parent link="base_link"/>
     <child link="lifting_tray"/>
-    <origin rpy="0 0 0" xyz="-0.065 0 0.1"/>
+    <origin rpy="0 0 0" xyz="0.0 0 0.105"/>
     <axis xyz="0 0 1"/>
     <limit effort="100" lower="0" upper="0.04" velocity="1"/>
-  </joint>
-  <gazebo reference="lifting_tray">
+  </joint> -->
+  <!-- <gazebo reference="lifting_tray">
     <selfCollide>true</selfCollide>
     <mu1 value="0.1"/>
@@ -46,10 +46,12 @@
     <kd value="10000" />
     <fdir1 value="0 0 0"/>
-  </gazebo>
-  <link name="lifting_tray">
-    <inertial>
-      <mass value="0.1"/>
+  </gazebo> -->
+  <!-- <link name="lifting_tray">
+    <inertial>
+      <mass value="2.8498940e-02"/>
       <origin rpy="0  0  0" xyz="0 0 0"/>
-      <inertia ixx="1" ixy="0" ixz="0" iyy="1" iyz="0" izz="1"/>
+      <inertia ixx="1.1175580e-05" ixy="-4.2369783e-11" ixz="-5.9381719e-09"
+               iyy="1.1192413e-05" iyz="-1.4400107e-11"
+               izz="2.0712558e-05"/>
     </inertial>
     <collision name="lifting_tray_collision">
@@ -65,5 +67,5 @@
       </geometry>
     </visual>
-  </link> -->
+  </link>  -->
   <joint name="wheel_left_joint" type="continuous">
     <parent link="base_link"/>
@@ -71,5 +73,14 @@
     <origin xyz="0.0 0.144 0.023" rpy="-1.57 0 0"/>
     <axis xyz="0 0 1"/>
-  </joint>
+    <limit effort="-1.0" lower="-1e+16" upper="1e+16" velocity="-1.0"/>
+  </joint>
+  <gazebo reference="wheel_left_link">
+    <selfCollide>false</selfCollide>
+    <mu1 value="100"/>
+    <mu2 value="50"/>
+    <kp value="10000000.0" />
+    <kd value="1000" />
+    <fdir1 value="0 0 0"/>
+  </gazebo>
   <link name="wheel_left_link">
     <visual>
@@ -87,4 +98,9 @@
     </collision>
     <inertial>
+      <!-- <origin xyz="0 0 0" />
+      <mass value="1" />
+      <inertia ixx="1" ixy="0" ixz="0"
+               iyy="1" iyz="0"
+               izz="1" /> -->
       <origin xyz="0 0 0" />
       <mass value="2.8498940e-02" />
@@ -94,4 +110,12 @@
       </inertial>
   </link>
+  <gazebo reference="right_wheel">
+    <selfCollide>false</selfCollide>
+    <mu1 value="100"/>
+    <mu2 value="50"/>
+    <kp value="10000000.0" />
+    <kd value="1000" />
+    <fdir1 value="0 0 0"/>
+  </gazebo>
   <joint name="wheel_right_joint" type="continuous">
     <parent link="base_link"/>
@@ -99,4 +123,5 @@
     <origin xyz="0.0 -0.144 0.023" rpy="-1.57 0 0"/>
     <axis xyz="0 0 1"/>
+    <limit effort="-1.0" lower="-1e+16" upper="1e+16" velocity="-1.0"/>
   </joint>
   <link name="wheel_right_link">
@@ -122,4 +147,32 @@
       </inertial>
   </link>
+  <!-- <joint name="wheel_front_joint" type="continuous">
+    <parent link="base_link"/>
+    <child link="wheel_front_link"/>
+    <origin xyz="0.1 0 0.023" rpy="-1.57 0 0"/>
+    <axis xyz="0 0 1"/>
+  </joint>
+  <link name="wheel_front_link">
+    <visual>
+      <origin xyz="0 0 0" rpy="1.57 0 0"/>
+      <geometry>
+        <mesh filename="package://turtlebot3_description/meshes/wheels/right_tire.stl" scale="0.001 0.001 0.001"/>
+      </geometry>
+      <material name="dark"/>
+    </visual>
+    <collision>
+      <origin xyz="0 0 0" rpy="0 0 0"/>
+      <geometry>
+        <cylinder length="0.018" radius="0.033"/>
+      </geometry>
+    </collision>
+    <inertial>
+      <origin xyz="0 0 0" />
+      <mass value="2.8498940e-02" />
+      <inertia ixx="1.1175580e-05" ixy="-4.2369783e-11" ixz="-5.9381719e-09"
+               iyy="1.1192413e-05" iyz="-1.4400107e-11"
+               izz="2.0712558e-05" />
+      </inertial>
+  </link> -->
   <joint name="caster_back_right_joint" type="fixed">
     <parent link="base_link"/>
@@ -127,4 +180,32 @@
     <origin xyz="-0.177 -0.064 -0.004" rpy="-1.57 0 0"/>
   </joint>
+  <!-- <joint name="wheel_behind_joint" type="continuous">
+    <parent link="base_link"/>
+    <child link="wheel_behind_link"/>
+    <origin xyz="-0.25 0.0 0.023" rpy="-1.57 0 0"/>
+    <axis xyz="0 0 1"/>
+  </joint>
+  <link name="wheel_behind_link">
+    <visual>
+      <origin xyz="0 0 0" rpy="1.57 0 0"/>
+      <geometry>
+        <mesh filename="package://turtlebot3_description/meshes/wheels/right_tire.stl" scale="0.001 0.001 0.001"/>
+      </geometry>
+      <material name="dark"/>
+    </visual>
+    <collision>
+      <origin xyz="0 0 0" rpy="0 0 0"/>
+      <geometry>
+        <cylinder length="0.018" radius="0.033"/>
+      </geometry>
+    </collision>
+    <inertial>
+      <origin xyz="0 0 0" />
+      <mass value="2.8498940e-02" />
+      <inertia ixx="1.1175580e-05" ixy="-4.2369783e-11" ixz="-5.9381719e-09"
+               iyy="1.1192413e-05" iyz="-1.4400107e-11"
+               izz="2.0712558e-05" />
+      </inertial>
+  </link> -->
   <link name="caster_back_right_link">
     <collision>
@@ -238,35 +319,3 @@
   </joint>
   <link name="camera_rgb_optical_frame"/>
-  <gazebo reference="laser">
-    <material>Gazebo/FlatBlack</material>
-    <sensor type="ray" name="lds_lfcd_sensor">
-      <pose>0 0 0 0 0 0</pose>
-      <visualize>false</visualize>
-      <update_rate>5</update_rate>
-      <ray>
-        <scan>
-          <horizontal>
-            <samples>360</samples>
-            <resolution>1</resolution>
-            <min_angle>0.0</min_angle>
-            <max_angle>6.28319</max_angle>
-          </horizontal>
-        </scan>
-        <range>
-          <min>0.120</min>
-          <max>10.0</max>
-          <resolution>0.050</resolution>
-        </range>
-        <noise>
-          <type>gaussian</type>
-          <mean>0.0</mean>
-          <stddev>0.01</stddev>
-        </noise>
-      </ray>
-      <plugin name="gazebo_ros_lds_lfcd_controller" filename="libgazebo_ros_laser.so">
-        <topicName>scan</topicName>
-        <frameName>laser</frameName>
-      </plugin>
-    </sensor>
-  </gazebo>
 </robot>

File: warehouse_simulation_toolkit/urdf/pioneer3dx_body.xacro (robot description, xacro)
@@ -2,4 +2,10 @@
 <robot xmlns:xacro="http://ros.org/wiki/xacro">
   <xacro:include filename="$(find warehouse_simulation)/urdf/pioneer3dx_wheel.xacro"/>
+  <link name="base_footprint"/>
+  <joint name="base_joint" type="fixed">
+    <parent link="base_footprint"/>
+    <child link="base_link" />
+    <origin xyz="0 0 0.010" rpy="0 0 0"/>
+  </joint>
   <!-- Chassis description -->
   <link name="base_link">
