Commit message: 

File: Warehouse_Gazebo/robot_description/urdf/robot.urdf.xacro (robot description, xacro)
@@ -53,5 +53,5 @@
     <limit effort="-1.0" lower="-1e+16" upper="1e+16" velocity="-1.0"/>
   </joint>
-  <gazebo reference="base_link_2">
+  <!-- <gazebo reference="base_link_2">
     <selfCollide>true</selfCollide>
     <mu1 value="0.3"/>
@@ -60,5 +60,5 @@
     <kd value="1000" />
     <fdir1 value="0 0 0"/>
-  </gazebo>
+  </gazebo> -->
   <link name="base_link">
   </link>
@@ -78,5 +78,5 @@
       <origin rpy="0  0  3.14" xyz="0  0  0.0118"/>
       <geometry>
-        <mesh filename="package://robot_description/models/laser_robot/meshes/carcaca.dae" scale="1 1 1"/>
+        <mesh filename="package://robot_description/models/laser_robot/meshes/carcaca.dae" scale="0.7 0.7 0.7"/>
       </geometry>
     </collision>
@@ -84,9 +84,9 @@
       <origin rpy="0  0  3.14" xyz="0  0  0.0118"/>
       <geometry>
-        <mesh filename="package://robot_description/models/laser_robot/meshes/carcaca.dae" scale="1 1 1"/>
-      </geometry>
-    </visual>
-  </link>
-  <gazebo reference="wheel_front_left">
+        <mesh filename="package://robot_description/models/laser_robot/meshes/carcaca.dae" scale="0.99 0.99 0.99"/>
+      </geometry>
+    </visual>
+  </link>
+  <!-- <gazebo reference="wheel_front_left">
     <selfCollide>true</selfCollide>
     <mu1 value="0.09"/>
@@ -95,5 +95,5 @@
     <kd value="10000" />
     <fdir1 value="0 0 0"/>
-  </gazebo>
+  </gazebo> -->
   <link name="wheel_front_left">
     <inertial>
@@ -115,5 +115,5 @@
     </visual>
   </link>
-  <gazebo reference="wheel_rear_left">
+  <!-- <gazebo reference="wheel_rear_left">
     <selfCollide>true</selfCollide>
     <mu1 value="0.09"/>
@@ -122,5 +122,5 @@
     <kd value="10000" />
     <fdir1 value="0 0 0"/>
-  </gazebo>
+  </gazebo> -->
   <link name="wheel_rear_left">
     <inertial>
@@ -142,5 +142,5 @@
     </visual>
   </link>
-  <gazebo reference="wheel_front_right">
+  <!-- <gazebo reference="wheel_front_right">
     <selfCollide>true</selfCollide>
     <mu1 value="0.09"/>
@@ -149,5 +149,5 @@
     <kd value="10000" />
     <fdir1 value="0 0 0"/>
-  </gazebo>
+  </gazebo> -->
   <link name="wheel_front_right">
     <inertial>
@@ -169,5 +169,5 @@
     </visual>
   </link>
-  <gazebo reference="wheel_rear_right">
+  <!-- <gazebo reference="wheel_rear_right">
     <selfCollide>true</selfCollide>
     <mu1 value="0.09"/>
@@ -176,5 +176,5 @@
     <kd value="10000" />
     <fdir1 value="0 0 0"/>
-  </gazebo>
+  </gazebo> -->
   <link name="wheel_rear_right">
     <inertial>
@@ -196,5 +196,5 @@
     </visual>
   </link>
-  <gazebo reference="lifting_tray">
+  <!-- <gazebo reference="lifting_tray">
     <selfCollide>true</selfCollide>
     <mu1 value="0.1"/>
@@ -203,5 +203,5 @@
     <kd value="10000" />
     <fdir1 value="0 0 0"/>
-  </gazebo>
+  </gazebo> -->
   <link name="lifting_tray">
     <inertial>
@@ -213,5 +213,5 @@
       <origin rpy="0  0  0" xyz="0 0 0"/>
       <geometry>
-        <mesh filename="package://robot_description/models/laser_robot/meshes/lifting.dae" scale="1 1 1"/>
+        <mesh filename="package://robot_description/models/laser_robot/meshes/lifting.dae" scale="1.0 1.0 1.0"/>
       </geometry>
     </collision>
@@ -242,5 +242,5 @@
     </visual>
   </link>
-  <gazebo reference="left_wheel">
+  <!-- <gazebo reference="left_wheel">
     <selfCollide>false</selfCollide>
     <mu1 value="100"/>
@@ -249,5 +249,5 @@
     <kd value="1000" />
     <fdir1 value="0 0 0"/>
-  </gazebo>
+  </gazebo> -->
   <link name="left_wheel">
     <inertial>
@@ -269,5 +269,5 @@
     </visual>
   </link>
-  <gazebo reference="right_wheel">
+  <!-- <gazebo reference="right_wheel">
     <selfCollide>false</selfCollide>
     <mu1 value="100"/>
@@ -276,5 +276,5 @@
     <kd value="1000" />
     <fdir1 value="0 0 0"/>
-  </gazebo>
+  </gazebo> -->
   <link name="right_wheel">
     <inertial>
@@ -360,10 +360,10 @@
       <material name="dark"/>
     </visual>
-    <collision>
+    <!-- <collision>
       <origin xyz="0.015 0 -0.0065" rpy="0 0 0"/>
       <geometry>
         <cylinder length="0.0315" radius="0.055"/>
       </geometry>
-    </collision>
+    </collision> -->
     <inertial>
       <mass value="0.114" />
